File: Hardware/v2 - RP2040/Nixie Clock v2/MCU.kicad_sch (KiCad schematic)
At the start: 29 parts, among them J1 USB_C_Receptacle_USB2.0, J2 Conn_01x03, J3 Conn_01x03, SW1 SW_Push, SW2 SW_Push, U1 RP2040, U2 W25Q128JVP, Y1 12MHz

Commit message: Complteted schematic, mergerd schematic on to one sheet, started assigning footprints
Parts:
- added BT1: CR1220, symbol Device:Battery_Cell
- added C11 (x5): 1u, symbol Device:C_Small
- added C11 (x4), C2 (x5): 100n, symbol Device:C_Small
- added C11: 10n, symbol Device:C_Small
- added C11, C2: 10u, symbol Device:C_Small
- added C14: 100u, symbol Device:C_Small
- added C15: 4.7u, symbol Device:C_Polarized_Small_US
- added C2: 33n, symbol Device:C_Small
- added C2: 82p, symbol Device:C_Small
- added C2: 47u, symbol Device:C_Small
- added J4: Conn_02x02_2.54mm, symbol Connector_Generic:Conn_02x02_Odd_Even
- added JP1, JP2: SolderJumper_2_Open, symbol Jumper:SolderJumper_2_Open
- added L1: 7.8u, symbol Device:L
- added N1, N2, N3, N4: ИN-8, symbol 0_My_Symbols:ИN-8
- added Q1, Q3: PZTA92, Package_TO_SOT_SMD:SOT-223-3_TabPin2, symbol Transistor_BJT:PZTA92
- added Q2, Q4: MMBTA42, Package_TO_SOT_SMD:SOT-23, symbol Transistor_BJT:MMBTA42
- added R10, R15, R16, R26, R27, R28, R29, R30, R31, R6: 10k, symbol Device:R_Small_US
- added R11: 150, symbol Device:R_Small_US
- added R12, R13, R14, R23, R24, R25: 100k, symbol Device:R_Small_US
- added R17, R18, R19, R20: 22k, symbol Device:R_Small_US
- added R21, R22: 220k, symbol Device:R_Small_US
- added R6: 30.9, symbol Device:R_Small_US
- added R9: R_Photo, symbol Device:R_Photo
- added SW1: SW_Push, symbol Switch:SW_Push
- added SW3: SW_DIP_x10, symbol Switch:SW_DIP_x10
- added U10: 74LVC1GU04DRL, Package_TO_SOT_SMD:SOT-553, symbol 74xGxx:74LVC1GU04DRL
- added U11: L80-M39, symbol 0_My_Symbols:L80-M39
- added U12: TPS62933, Package_TO_SOT_SMD:SOT-583-8, symbol Regulator_Switching:TPS62933
- added U13: TC2185-3.3VCTTR, Package_TO_SOT_SMD:SOT-23-5, symbol Regulator_Linear:TC2185-3.3VxCTTR
- added U14: AP22913, symbol 0_My_Symbols:AP22913
- added U3, U4, U5, U6: К155ИД1, symbol 0_My_Symbols:К155ИД1
- added U7: NCH8200HV, symbol 0_My_Symbols:NCH8200HV
- added U8: MCP23017_SO, Package_SO:SOIC-28W_7.5x17.9mm_P1.27mm, symbol Interface_Expansion:MCP23017_SO
- added U9: DS3231MZ, Package_SO:SOIC-8_3.9x4.9mm_P1.27mm, symbol Timer_RTC:DS3231MZ
- J2, J3: value Conn_01x03 -> Conn_01x03_2.54mm
Connections:
- net Dimming_2 is gone; now on net GPS_EN: U1.35 (GPIO23)
- net +3.3V: now also C2.1, C2.1, L1.2, R6.2, U10.5 (VCC)
- net +3V3: now also C11.1, C11.1, C11.1, R28.1, R29.1, R30.1, U14.4 (VIN), U14.6 (VIN), U8.9 (VDD), U9.2 (VCC), U9.4 (~{RST})
- net GND: now also BT1.2 (-), C11.2, C11.2, C11.2, C11.2, C11.2, C11.2, C11.2, C11.2, C11.2, C11.2, C11.2, C14.2, C15.2, C2.2, C2.2, C2.2, C2.2, C2.2, C2.2, C2.2, J4.1 (Pin_1), J4.3 (Pin_3), Q2.2 (E), Q4.2 (E), R10.2, R16.2, R27.2, R6.1, SW3.11, SW3.12, SW3.13, SW3.14, SW3.15, SW3.16, SW3.17, SW3.18, SW3.19, SW3.20, U10.3 (GND), U11.12 (GND), U11.3 (GND), U11.7 (TIMER), U12.4 (GND), U13.2 (GND), U14.2 (GND), U14.5 (GND), U3.12 (GND), U4.12 (GND), U5.12 (GND), U6.12 (GND), U7.2 (GND), U7.4 (GND), U8.10 (VSS), U8.15 (A0), U8.16 (A1), U8.17 (A2), U9.5 (GND)
- net GPS_EN: now also U14.3 (EN); no longer U1.36 (GPIO24)
- net Hours_Ones_A: now also U4.3 (A)
- net Hours_Ones_B: now also U4.6 (B)
- net Hours_Ones_C: now also U4.7 (C)
- net Hours_Ones_D: now also U4.4 (D)
- net Hours_Tens_A: now also U3.3 (A)
- net Hours_Tens_B: now also U3.6 (B)
- net Hours_Tens_C: now also U3.7 (C)
- net Hours_Tens_D: now also U3.4 (D)
- net I2C0 SCL: now also U8.12 (SCK), U9.8 (SCL)
- net Light: now also U1.38 (GPIO26_ADC0), C11.1, R11.2; no longer U1.39 (GPIO27_ADC1)
- net Mins_Ones_A: now also U6.3 (A)
- net Mins_Ones_B: now also U6.6 (B)
- net Mins_Ones_C: now also U6.7 (C)
- net Mins_Ones_D: now also U6.4 (D)
- net Mins_Tens_A: now also U5.3 (A)
- net Mins_Tens_B: now also U5.6 (B)
- net Mins_Tens_C: now also U5.7 (C)
- net Mins_Tens_D: now also U5.4 (D)
- net RTC_Interrupt: now also U1.36 (GPIO24), U9.3 (~{INT}/SQW); no longer U1.38 (GPIO26_ADC0)
- net Settings_Interrupt: now also R29.2, U8.20 (INTA)
- net VBUS: now also C11.1, C14.1, C2.1, C2.1, U12.3 (VIN), U13.1 (VIN), U13.3 (ON/~{OFF}), U3.5 (Vcc), U4.5 (Vcc), U5.5 (Vcc), U6.5 (Vcc), U7.1 (Vin)
- net at R7.1, R8.2, SW1.2: now also C2.1
- net at R6.1, SW2.2, U1.26 (RUN): now also C2.1
- net Dimming_1 renamed Dimming
- net Dimming: now also R15.1, R16.1, U10.2
- net I2C0 SDA renamed I2C0_SDA
- net I2C0_SDA: now also U8.13 (SDA), U9.7 (SDA)
- net UART1 RX renamed UART1_RX
- net UART1_RX: now also U11.2 (TXD1)
- net UART1 TX renamed UART1_TX
- net UART1_TX: now also U11.1 (RXD1)
- new net: JP1.1 (A), Q1.2 (C), R17.1, R18.1, R21.1
- new net: N1.11 (Anode), R17.2
- new net: C2.2, R6.1, R6.2, U12.8 (FB)
- new net: C2.1, U12.7 (SS)
- new net: SW3.1, U8.1 (GPB0)
- new net: R28.2, U8.18 (~{RESET})
- new net: R30.2, U8.19 (INTB)
- new net: SW3.2, U8.2 (GPB1)
- new net: SW3.9, U8.21 (GPA0)
- new net: SW3.10, U8.22 (GPA1)
- new net: SW1.1, U8.23 (GPA2)
- new net: SW3.3, U8.3 (GPB2)
- new net: SW3.4, U8.4 (GPB3)
- new net: SW3.5, U8.5 (GPB4)
- new net: SW3.6, U8.6 (GPB5)
- new net: SW3.7, U8.7 (GPB6)
- new net: SW3.8, U8.8 (GPB7)
- new net: C11.1, C11.1, C11.1, C11.1, R31.1, U11.4 (VCC), U11.5 (V_BCKP), U14.1 (OUT)
- new net: JP1.2 (B), Q3.2 (C), R19.1, R20.1, R22.1
- new net: N3.11 (Anode), R19.2
- new net: N1.1, U3.15 (1)
- new net: N1.10 (0), U3.16 (0)
- new net: N1.2, U3.8 (2)
- new net: N1.3, U3.9 (3)
- new net: N1.4, U3.13 (4)
- new net: N1.5, U3.14 (5)
- new net: N1.6, U3.11 (6)
- new net: N1.7, U3.10 (7)
- new net: N1.8, U3.1 (8)
- new net: N1.9, U3.2 (9)
- new net: C2.1, SW1.2
- new net: N4.1, U6.15 (1)
- new net: N4.10 (0), U6.16 (0)
- new net: N4.11 (Anode), R20.2
- new net: N4.2, U6.8 (2)
- new net: N4.3, U6.9 (3)
- new net: N4.4, U6.13 (4)
- new net: N4.5, U6.14 (5)
- new net: N4.6, U6.11 (6)
- new net: N4.7, U6.10 (7)
- new net: N4.8, U6.1 (8)
- new net: N4.9, U6.2 (9)
- new net: R26.1, R27.1, U10.4
- new net: Q1.1 (B), R12.2, R13.1
- new net: R13.2, R14.1
- new net: C11.1, U13.4 (BP)
- new net: R24.2, R25.1
- new net: Q4.3 (C), R25.2
- new net: Q4.1 (B), R26.2
- new net: Q2.1 (B), R15.2
- new net: BT1.1 (+), U9.6 (VBAT)
- new net: J4.4 (Pin_4), R22.2
- new net: C15.1, JP2.1 (A), Q1.3 (E), R12.1, U7.3 (170V)
- new net: JP2.2 (B), Q3.3 (E), R23.1
- new net: Q3.1 (B), R23.2, R24.1
- new net: N3.1, U5.15 (1)
- new net: N3.10 (0), U5.16 (0)
- new net: N3.2, U5.8 (2)
- new net: N3.3, U5.9 (3)
- new net: N3.4, U5.13 (4)
- new net: N3.5, U5.14 (5)
- new net: N3.6, U5.11 (6)
- new net: N3.7, U5.10 (7)
- new net: N3.8, U5.1 (8)
- new net: N3.9, U5.2 (9)
- new net: Q2.3 (C), R14.2
- new net: R31.2, U11.10 (~{RESET})
- new net: N2.11 (Anode), R18.2
- new net: N2.1, U4.15 (1)
- new net: N2.10 (0), U4.16 (0)
- new net: N2.2, U4.8 (2)
- new net: N2.3, U4.9 (3)
- new net: N2.4, U4.13 (4)
- new net: N2.5, U4.14 (5)
- new net: N2.6, U4.11 (6)
- new net: N2.7, U4.10 (7)
- new net: N2.8, U4.1 (8)
- new net: N2.9, U4.2 (9)
- new net: C2.2, L1.1, U12.5 (SW)
- new net: C2.1, U12.6 (BST)
- new net: R10.1, R11.1, R9.2
- new net: J4.2 (Pin_2), R21.2
- new net +3.3VA: C11.1, R9.1, U13.5 (VOUT)
- no-connect marks 2 -> 11
Other:
- note added: "1060Hz LPF Sample at <= 530Hz or 1.89ms"
- note added: "219-10MST"
- note added: "250V or larger"
- note added: "Close either JP1 OR JP2, NOT BOTH. Close JP1 for 1 switching circuit Close JP2 for 2 switching circuits"
- note added: "Colon mounting point"
- note added: "DNP Might be needed to balance load on power supply"
- note added: "Linear supply for analog circuits"
- note added: "Low ESR"
- note added: "Vin to 3.3V"
- moved on the sheet: C1, C10, C11, C12, C13, C2, C3, C4, C5, C6, C7, C8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
