File: Hardware/v2 - RP2040/Nixie Clock v2/Nixie Clock v2.kicad_pcb (KiCad board)
At the start: 2 copper layers, 100 x 100 mm, 105 parts, among them J1 Conn_02x02_2.54mm, J2 USB_C_Receptacle_USB2.0, J3 Conn_01x03_2.54mm, J4 Conn_01x03_2.54mm, Q1 PZTA92, Q2 PZTA92, Q3 MMBTA42, Q4 MMBTA42, SW1 SW_Push, SW2 SW_Push, SW3 SW_DIP_x10, SW4 SW_Push, U1 NCH8200HV, U10 W25Q128JVP, U11 L80-M39, U12 DS3231MZ, U13 TC2185-3.3VCTTR, U14 MCP23017_SS, U2 74LVC1GU04DRL, U3 TPS62933, U4 К155ИД1, U5 К155ИД1, U6 К155ИД1, U7 К155ИД1, U8 AP22913, U9 RP2040, Y1 12MHz

Commit message: Continued work on layout
Parts:
- moved R28 392.3 mm to (176.0, 358.5)
- moved R29 392.3 mm to (176.0, 361.0)
- moved C1 386.0 mm to (213.8, 276.8)
- moved R34 385.1 mm to (-4.00, 421.5)
- moved R33 384.9 mm to (-8.50, 419.5)
- moved R35 384.0 mm to (-8.00, 423.5)
- moved C34 381.9 mm to (-3.00, 426.0)
- moved C31 381.8 mm to (3.36, 417.0)
- moved C32 381.8 mm to (3.36, 419.6)
- moved C30 381.8 mm to (3.36, 414.5)
- moved J3 376.5 mm to (152.1, 370.1)
- moved J4 376.5 mm to (156.7, 370.1)
- moved C11 372.8 mm to (139.8, 351.8)
- moved C12 372.8 mm to (143.9, 329.3)
- moved C14 372.8 mm to (143.9, 334.3)
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Connections:
- net Net-(JP1-A) renamed /170V_1
- net Net-(JP1-B) renamed /170V_2
- net Net-(JP2-A) renamed /ANODE_1
- net Net-(JP2-B) renamed /ANODE_2
- C35 pad 1: GND -> Net-(U14-GPA2)
Routing:
- net /170V_1: track 0.00 -> 0.95 mm
- net Net-(Q1-B): track 0.00 -> 0.88 mm

Commit message: replaced old nixie compontes with new library and replaced IO expander with QFN
Parts:
- removed JP1, JP2: SolderJumper_2_Open, Jumper:SolderJumper-2_P1.3mm_Open_TrianglePad1.0x1.5mm
- removed N1, N2, N3, N4: ИN-8, Display_Nixie:ИN-8 DSUB
- removed Q2: PZTA92, Package_TO_SOT_SMD:SOT-223-3_TabPin2
- removed Q4: MMBTA42, Package_TO_SOT_SMD:SOT-23
- removed R10, R8: 10k, Resistor_SMD:R_0603_1608Metric
- removed R2, R4, R6: 100k, Resistor_SMD:R_0603_1608Metric
- removed U1: NCH8200HV, Display_Nixie:NCH8200HV
- removed U2: 74LVC1GU04DRL, Package_TO_SOT_SMD:SOT-553
- removed the U7 at (194.1, 124.2)
- removed Y1: 12MHz, 0_My_Footprints:Crystal_SMD_Abracon_ABM10-4Pin_2.5x2.0mm
- added U7: MCP23017_ML, Package_DFN_QFN:QFN-28-1EP_6x6mm_P0.65mm_EP4.25x4.25mm, F.Cu at (-39.2, -10.9)
- added U7: К155ИД1, Package_DIP:DIP-16_W7.62mm, F.Cu at (-45.7, 31.9)
- BT1, C2, L1: moved to B.Cu
- moved R29 429.4 mm to (-61.8, 3.42)
- moved C34 413.0 mm to (-69.8, 18.5)
- moved C31 412.6 mm to (-69.8, 10.9)
- moved C32 412.6 mm to (-69.8, 13.5)
- moved C30 412.6 mm to (-69.8, 8.44)
- moved R34 409.6 mm to (-61.8, 16.0)
- moved R33 409.5 mm to (-61.8, 13.5)
- moved R28 409.1 mm to (-65.8, 28.5)
- moved R35 408.6 mm to (-61.8, 18.5)
- moved J3 406.2 mm to (-57.5, 22.0)
- moved J4 406.2 mm to (-52.8, 22.0)
- moved C18 402.5 mm to (-88.9, 58.7)
- moved C27 402.5 mm to (-88.9, 62.6)
- moved C19 402.5 mm to (-88.9, 60.7)
- moved C28 402.5 mm to (-88.9, 64.6)
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Connections:
- C35 pad 1: Net-(U14-GPA2) -> Net-(U7-GPA2)
- R14 pad 1: /ANODE_2 -> /ANODE_1
- R15 pad 1: /ANODE_2 -> /ANODE_1
- R16 pad 1: /ANODE_2 -> /ANODE_1
- R31 pad 2: Net-(U14-INTB) -> Net-(U7-INTB)
- R32 pad 2: Net-(U14-~{RESET}) -> Net-(U7-~{RESET})
- SW3 pad 1: Net-(U14-GPB0) -> Net-(U7-GPB0)
- SW3 pad 10: Net-(U14-GPA1) -> Net-(U7-GPA1)
- SW3 pad 2: Net-(U14-GPB1) -> Net-(U7-GPB1)
- SW3 pad 3: Net-(U14-GPB2) -> Net-(U7-GPB2)
- SW3 pad 4: Net-(U14-GPB3) -> Net-(U7-GPB3)
- SW3 pad 5: Net-(U14-GPB4) -> Net-(U7-GPB4)
- SW3 pad 6: Net-(U14-GPB5) -> Net-(U7-GPB5)
- SW3 pad 7: Net-(U14-GPB6) -> Net-(U7-GPB6)
- SW3 pad 8: Net-(U14-GPB7) -> Net-(U7-GPB7)
- SW3 pad 9: Net-(U14-GPA0) -> Net-(U7-GPA0)
- SW4 pad 1: Net-(U14-GPA2) -> Net-(U7-GPA2)
Routing:
- net /170V_1: track 0.95 -> 0.00 mm
- net Net-(Q1-B): track 0.88 -> 0.00 mm
