File: Hardware/v2 - RP2040/Nixie Clock v2/Nixie Clock v2.kicad_sch (KiCad schematic)
At the start: 105 parts, among them J1 Conn_02x02_2.54mm, J2 USB_C_Receptacle_USB2.0, J3 Conn_01x03_2.54mm, J4 Conn_01x03_2.54mm, Q1 PZTA92, Q2 PZTA92, Q3 MMBTA42, Q4 MMBTA42, SW1 SW_Push, SW2 SW_Push, SW3 SW_DIP_x10, SW4 SW_Push, U1 NCH8200HV, U10 W25Q128JVP, U11 L80-M39, U12 DS3231MZ, U13 TC2185-3.3VCTTR, U14 MCP23017_SS, U2 74LVC1GU04DRL, U3 TPS62933, U4 К155ИД1, U5 К155ИД1, U6 К155ИД1, U7 К155ИД1, U8 AP22913, U9 RP2040, Y1 12MHz

Commit message: replaced old nixie compontes with new library and replaced IO expander with QFN
Parts:
- removed JP1, JP2: SolderJumper_2_Open, Jumper:SolderJumper-2_P1.3mm_Open_TrianglePad1.0x1.5mm, symbol Jumper:SolderJumper_2_Open
- removed N1, N2, N3, N4: ИN-8, Display_Nixie:ИN-8 DSUB, symbol 0_My_Symbols:ИN-8
- removed Q2: PZTA92, Package_TO_SOT_SMD:SOT-223-3_TabPin2, symbol Transistor_BJT:PZTA92
- removed Q4: MMBTA42, Package_TO_SOT_SMD:SOT-23, symbol Transistor_BJT:MMBTA42
- removed R10, R8: 10k, Resistor_SMD:R_0603_1608Metric, symbol Device:R_Small_US
- removed R2, R4, R6: 100k, Resistor_SMD:R_0603_1608Metric, symbol Device:R_Small_US
- removed U1: NCH8200HV, Display_Nixie:NCH8200HV, symbol 0_My_Symbols:NCH8200HV
- removed U14: MCP23017_SS, Package_SO:SSOP-28_5.3x10.2mm_P0.65mm, symbol Interface_Expansion:MCP23017_SS
- removed U2: 74LVC1GU04DRL, Package_TO_SOT_SMD:SOT-553, symbol 74xGxx:74LVC1GU04DRL
- removed U4, U5, U6, U7: К155ИД1, Package_DIP:DIP-16_W7.62mm, symbol 0_My_Symbols:К155ИД1
- added N1, N2, N3, N4: ИN-8, symbol Nick-Nixie:ИN-8
- added U1: NCH8200HV, symbol Nick-Nixie:NCH8200HV
- added U2, U4, U5, U6: К155ИД1, symbol Nick-Nixie:К155ИД1
- added U7: MCP23017_ML, Package_DFN_QFN:QFN-28-1EP_6x6mm_P0.65mm_EP4.25x4.25mm, symbol Interface_Expansion:MCP23017_ML
Connections:
- net ANODE_2 is gone; now on net ANODE_1: R14.1, R15.1, R16.1
- net +3V3: now also U7.5 (VDD)
- net 170V_1: now also U1.3 (170V)
- net GND: now also U1.2 (GND), U1.4 (GND), U2. (Vcc), U4. (Vcc), U5. (Vcc), U6. (Vcc), U7.11 (A0), U7.12 (A1), U7.13 (A2), U7.29 (EP), U7.6 (VSS)
- net Hours_Ones_A: now also U4. (Vcc)
- net Hours_Ones_B: now also U4. (Vcc)
- net Hours_Ones_C: now also U4. (Vcc)
- net Hours_Ones_D: now also U4. (Vcc)
- net Hours_Tens_A: now also U2. (Vcc)
- net Hours_Tens_B: now also U2. (Vcc)
- net Hours_Tens_C: now also U2. (Vcc)
- net Hours_Tens_D: now also U2. (Vcc)
- net I2C0 SCL: now also U7.8 (SCK)
- net I2C0_SDA: now also U7.9 (SDA)
- net Mins_Ones_A: now also U6. (Vcc)
- net Mins_Ones_B: now also U6. (Vcc)
- net Mins_Ones_C: now also U6. (Vcc)
- net Mins_Ones_D: now also U6. (Vcc)
- net Mins_Tens_A: now also U5. (Vcc)
- net Mins_Tens_B: now also U5. (Vcc)
- net Mins_Tens_C: now also U5. (Vcc)
- net Mins_Tens_D: now also U5. (Vcc)
- net Settings_Interrupt: now also U7.16 (INTA)
- net VBUS: now also U1.1 (Vin), U2. (Vcc), U4. (Vcc), U5. (Vcc), U6. (Vcc)
- net at C35.1, SW4.1: now also U7.19 (GPA2)
- net at R12.2: now also N2.11 (Anode)
- net at R11.2: now also N1.11 (Anode)
- net at R16.2: now also N4.11 (Anode)
- net at SW3.1: now also U7.25 (GPB0)
- net at SW3.10: now also U7.18 (GPA1)
- net at SW3.2: now also U7.26 (GPB1)
- net at SW3.3: now also U7.27 (GPB2)
- net at SW3.4: now also U7.28 (GPB3)
- net at SW3.5: now also U7.1 (GPB4)
- net at SW3.6: now also U7.2 (GPB5)
- net at SW3.7: now also U7.3 (GPB6)
- net at SW3.8: now also U7.4 (GPB7)
- net at SW3.9: now also U7.17 (GPA0)
- net at R31.2: now also U7.15 (INTB)
- net at R32.2: now also U7.14 (~{RESET})
- net at R15.2: now also N3.11 (Anode)
- new net: N3. (5), U5.14 (5)
- new net: N3.1, U5.15 (1)
- new net: N3.10 (0), U5.16 (0)
- new net: N3.2, U5.8 (2)
- new net: N3.3, U5.9 (3)
- new net: N3.4, U5.13 (4)
- new net: N3.6, U5.11 (6)
- new net: N3.7, U5.10 (7)
- new net: N3.8, U5.1 (8)
- new net: N3.9, U5. (Vcc)
- new net: N4.9, U6. (Vcc)
- new net: N4.8, U6.1 (8)
- new net: N4.7, U6.10 (7)
- new net: N4.6, U6.11 (6)
- new net: N4.4, U6.13 (4)
- new net: N4. (5), U6.14 (5)
- new net: N4.1, U6.15 (1)
- new net: N4.10 (0), U6.16 (0)
- new net: N4.2, U6.8 (2)
- new net: N4.3, U6.9 (3)
- new net: N1. (5), U2.14 (5)
- new net: N1.1, U2.15 (1)
- new net: N1.10 (0), U2.16 (0)
- new net: N1.2, U2.8 (2)
- new net: N1.3, U2.9 (3)
- new net: N1.4, U2.13 (4)
- new net: N1.6, U2.11 (6)
- new net: N1.7, U2.10 (7)
- new net: N1.8, U2.1 (8)
- new net: N1.9, U2. (Vcc)
- new net: N2. (5), U4.14 (5)
- new net: N2.1, U4.15 (1)
- new net: N2.10 (0), U4.16 (0)
- new net: N2.2, U4.8 (2)
- new net: N2.3, U4.9 (3)
- new net: N2.4, U4.13 (4)
- new net: N2.6, U4.11 (6)
- new net: N2.7, U4.10 (7)
- new net: N2.8, U4.1 (8)
- new net: N2.9, U4. (Vcc)
Other:
- note removed: "Close either JP1 OR JP2, NOT BOTH. Close JP1 for 1 switching circuit Close JP2 for 2 switching circuits"
- note removed: "DNP Might be needed to balance load on power supply"
